File: schematic/mosfet+buck_inverterV2.sch (EAGLE design)
At the start: 35 parts, among them IC2 ACS712-LC, K1 ZF112, K2 ZF112, Q5 BC847, Q6 IRF3205, Q7 BC847, Q8 BC847

Commit message: edit
Parts:
- added 220-, LOAD-: MKDSN1,5/2-5,08, con-phoenix-508:MKDSN1,5/2-5,08
- renumbered VIN+1 to 220+, VIN+2 to LOAD+
Connections:
- net N$20 renamed +24V_UNPROTECTED
- new net +48V: F1.2, JP3.1, JP3.2, JP3.3, R1.2, U$1.IN+
- new net +5V_PROTECTED: JP2.3, JP2.4, K12.P
- new net 220: 220--1.KL, 220--2.KL, LOAD--1.KL, LOAD--2.KL
- net +24V: no longer F1.2, JP3.1, JP3.2, JP3.3, R1.2, U$1.IN+
- net +5V: no longer JP2.3, JP2.4, K12.P
- net BAT_PROTECTED_GND: now also JP3.4, JP3.5, JP3.6
- net GND: no longer JP3.4, JP3.5, JP3.6
